File: drone-esc.kicad_sch (KiCad schematic)
At the start: 44 parts, among them J1 SM08B-SRSS-TB_LF__SN_, U2 INA186A3IDCKR, U3 TLV76733DRVR, U4 TPS61023DRLR

Commit message: added board footprint
Parts:
- R2: footprint Resistor_SMD:R_2512_6332Metric -> Resistor_SMD:R_0201_0603Metric
- U1: footprint (none) -> esc-board-copper:esc-board
Changed lines of the file:
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@@
 			)
 		)
-		(property "Footprint" "Resistor_SMD:R_2512_6332Metric"
+		(property "Footprint" "Resistor_SMD:R_0201_0603Metric"
 			(at 86.36 164.338 90)
 			(hide yes)
@@
 			)
 		)
-		(property "Footprint" ""
+		(property "Footprint" "esc-board-copper:esc-board"
 			(at 73.66 49.53 0)
 			(hide yes)

Commit message: basic placement 1
Parts:
- removed C11, C15, C20, C23: 10u, Capacitor_SMD:C_0805_2012Metric, symbol Device:C
Connections:
- net +BATT: no longer U1.3 (VBAT+)
- net CURR: no longer U1.5 (CUR)
- net GND: now also J1.P1, J1.P2; no longer U1.4 (GND)
- net M1: no longer U1.7 (M1)
- net M2: no longer U1.8 (M2)
- net M3: no longer U1.9 (M3)
- net M4: no longer U1.10 (M4)
- no-connect marks 2 -> 1
Other:
- note added: "(~30 µF nominal per motor)"
- note removed: "(~40 µF nominal per motor)"
- moved on the sheet: D2, D3, R5, R90, TP14, TP15

Commit message: final final group and place
Parts:
- added TP28: 3V3, TestPoint:TestPoint_Pad_D1.0mm, symbol Connector:TestPoint
Connections:
- net +3.3V: now also TP28.1
Changed lines of the file:
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@@
 	)
 	(junction
+		(at 59.69 143.51)
+		(diameter 0)
+		(color 0 0 0 0)
+	)
+	(junction
 		(at 193.04 67.31)
 		(diameter 0)
@@
 	(wire
 		(pts
+			(xy 59.69 143.51) (xy 59.69 140.97)
+		)
+		(stroke
+			(width 0)
+			(type default)
+		)
+	)
+	(wire
+		(pts
 			(xy 224.79 44.45) (xy 227.33 44.45)
 		)
@@
 	(wire
 		(pts
-			(xy 59.69 154.94) (xy 59.69 140.97)
+			(xy 59.69 154.94) (xy 59.69 143.51)
 		)
 		(stroke
@@
 					(unit 1)
 				)
+			)
+		)
+	)
+	(symbol
+		(lib_id "Connector:TestPoint")
+		(at 59.69 143.51 270)
+		(unit 1)
+		(body_style 1)
+		(exclude_from_sim no)
+		(in_bom yes)
+		(on_board yes)
+		(in_pos_files yes)
+		(dnp no)
+		(property "Reference" "TP28"
+			(at 68.326 143.764 0)
+			(show_name no)
+			(do_not_autoplace no)
+			(effects
+				(font
+					(size 1.27 1.27)
+				)
+			)
+		)
+		(property "Value" "3V3"
+			(at 65.786 143.764 0)
+			(show_name no)
+			(do_not_autoplace no)
+			(effects
+				(font
+					(size 1.27 1.27)
+				)
+			)
+		)
+		(property "Footprint" "TestPoint:TestPoint_Pad_D1.0mm"
+			(at 59.69 148.59 0)
+			(hide yes)
+			(show_name no)
+			(do_not_autoplace no)
+			(effects
+				(font
+					(size 1.27 1.27)
+				)
+			)
+		)
+		(property "Datasheet" ""
+			(at 59.69 148.59 0)
+			(hide yes)
+			(show_name no)
+			(do_not_autoplace no)
+			(effects
+				(font
+					(size 1.27 1.27)
+				)
+			)
+		)
+		(property "Description" "test point"
+			(at 59.69 143.51 0)
+			(hide yes)
+			(show_name no)
+			(do_not_autoplace no)
+			(effects
+				(font
+					(size 1.27 1.27)
+				)
+			)
+		)
+		(pin "1"
+		)
+		(instances
+			(project "drone-esc"
+				(path "/f59ffce8-13f3-438d-8235-d53c820346a5"
+					(reference "TP28")
+					(unit 1)
+				)

Commit message: main placing
Connections:
- net ESC3/A: now also U1.19 (3A); no longer U1.17 (3A)
- net ESC3/C: now also U1.17 (3C); no longer U1.19 (3C)
- net ESC4/A: now also U1.22 (4A); no longer U1.20 (4A)
- net ESC4/C: now also U1.20 (4C); no longer U1.22 (4C)
Changed lines of the file:
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@@
 	(wire
 		(pts
+			(xy 116.84 57.15) (xy 121.92 57.15)
+		)
+		(stroke
+			(width 0)
+			(type default)
+		)
+	)
+	(wire
+		(pts
 			(xy 134.62 160.02) (xy 139.7 160.02)
 		)
@@
 	(wire
 		(pts
-			(xy 116.84 57.15) (xy 121.92 57.15)
-		)
-		(stroke
-			(width 0)
-			(type default)
-		)
-	)
-	(wire
-		(pts
 			(xy 196.85 111.76) (xy 215.9 111.76)
 		)
@@
 	(wire
 		(pts
+			(xy 116.84 67.31) (xy 121.92 67.31)
+		)
+		(stroke
+			(width 0)
+			(type default)
+		)
+	)
+	(wire
+		(pts
 			(xy 96.52 162.56) (xy 100.33 162.56)
 		)
@@
 	(wire
 		(pts
-			(xy 116.84 67.31) (xy 121.92 67.31)
-		)
-		(stroke
-			(width 0)
-			(type default)
-		)
-	)
-	(wire
-		(pts
 			(xy 237.49 134.62) (xy 237.49 140.97)
 		)
@@
 		(pin "18"
 		)
+		(pin "5"
+		)
+		(pin "6"
+		)
+		(pin "7"
+		)
+		(pin "8"
+		)
+		(pin "9"
+		)
+		(pin "10"
+		)
+		(pin "4"
+		)
+		(pin "3"
+		)
 		(instances
 			(project "drone-esc"
@@
 		)
 		(pin "A" output
-			(at 121.92 72.39 180)
+			(at 121.92 82.55 180)
 			(effects
 				(font
@@
 		)
 		(pin "C" output
-			(at 121.92 82.55 180)
+			(at 121.92 72.39 180)
 			(effects
 				(font
@@
 		)
 		(pin "A" output
-			(at 121.92 57.15 180)
+			(at 121.92 67.31 180)
 			(effects
 				(font
@@
 		)
 		(pin "C" output
-			(at 121.92 67.31 180)
+			(at 121.92 57.15 180)
 			(effects
 				(font
