File: ESC.kicad_sch (KiCad schematic)
At the start: 61 parts, among them Q1 IRLHS6242, Q2 IRLHS6242, Q3 IRLHS6242, Q4 IRLHS6242, Q5 IRLHS6242, Q6 IRLHS6242, U5 AT32F421G8U7, U6 DGD05473FNQ-7, U7 DGD05473FNQ-7, U8 DGD05473FNQ-7

Commit message: added board footprint
Parts:
- removed TP28: GBH, TestPoint:TestPoint_Pad_D1.0mm, symbol Connector:TestPoint
- removed TP32: GCH, TestPoint:TestPoint_Pad_D1.0mm, symbol Connector:TestPoint
- removed TP40: GBL, TestPoint:TestPoint_Pad_D1.0mm, symbol Connector:TestPoint
- removed TP44: GCL, TestPoint:TestPoint_Pad_D1.0mm, symbol Connector:TestPoint
- removed TP60: VBA, TestPoint:TestPoint_Pad_D1.0mm, symbol Connector:TestPoint
- removed TP64: VBB, TestPoint:TestPoint_Pad_D1.0mm, symbol Connector:TestPoint
- removed TP68: VBC, TestPoint:TestPoint_Pad_D1.0mm, symbol Connector:TestPoint
- removed TP72: FBC, TestPoint:TestPoint_Pad_D1.0mm, symbol Connector:TestPoint
- removed TP76: ESC_EN, TestPoint:TestPoint_Pad_D1.0mm, symbol Connector:TestPoint

Commit message: placement 2 (starting routing)
Connections:
- net A_LOW: now also U5.19 (PA9); no longer U5.15 (PB1)
- net B_HIGH: now also U5.18 (PA8); no longer U5.19 (PA9)
- net B_LOW: now also U5.15 (PB1); no longer U5.14 (PB0)
- net C_HIGH: now also U5.14 (PB0); no longer U5.18 (PA8)
- net ESC_EN: now also U5.23 (PA15); no longer U5.28 (PB7)
- net FBA: now also U5.24 (PB3); no longer U5.6 (PA0)
- net FBB: now also U5.11 (PA5); no longer U5.10 (PA4)
- net FBC: now also U5.10 (PA4); no longer U5.11 (PA5)
Changed lines of the file:
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@@
 	)
 	(no_connect
+		(at 86.36 33.02)
+	)
+	(no_connect
 		(at 88.9 69.85)
 	)
@@
 	)
 	(no_connect
+		(at 76.2 57.15)
+	)
+	(no_connect
 		(at 76.2 49.53)
 	)
@@
 	)
 	(no_connect
-		(at 99.06 33.02)
-	)
-	(no_connect
-		(at 96.52 33.02)
-	)
-	(no_connect
 		(at 59.69 170.18)
 	)
@@
 	(wire
 		(pts
-			(xy 86.36 24.13) (xy 86.36 33.02)
-		)
-		(stroke
-			(width 0)
-			(type default)
-		)
-	)
-	(wire
-		(pts
 			(xy 87.63 173.99) (xy 102.87 173.99)
 		)
@@
 	(wire
 		(pts
-			(xy 73.66 57.15) (xy 76.2 57.15)
-		)
-		(stroke
-			(width 0)
-			(type default)
-		)
-	)
-	(wire
-		(pts
 			(xy 118.11 130.81) (xy 118.11 129.54)
 		)
@@
 	(wire
 		(pts
+			(xy 99.06 24.13) (xy 99.06 33.02)
+		)
+		(stroke
+			(width 0)
+			(type default)
+		)
+	)
+	(wire
+		(pts
 			(xy 248.92 118.11) (xy 252.73 118.11)
 		)
@@
 	(wire
 		(pts
+			(xy 96.52 31.75) (xy 96.52 33.02)
+		)
+		(stroke
+			(width 0)
+			(type default)
+		)
+	)
+	(wire
+		(pts
 			(xy 171.45 125.73) (xy 171.45 128.27)
 		)
@@
 	)
 	(label "ESC_EN"
-		(at 86.36 24.13 180)
+		(at 99.06 24.13 90)
 		(effects
 			(font
 				(size 1.27 1.27)
 			)
-			(justify right bottom)
+			(justify left bottom)
 		)
 	)
@@
 	)
 	(label "FBA"
-		(at 73.66 57.15 180)
-		(effects
-			(font
-				(size 1.27 1.27)
-			)
-			(justify right bottom)
-		)
-	)
-	(label "FBA"
 		(at 196.85 48.26 180)
 		(effects
@@
 		)
 	)
-	(label "C_HIGH"
+	(label "B_HIGH"
 		(at 111.76 52.07 0)
 		(effects
@@
 		)
 	)
-	(label "B_LOW"
+	(label "C_HIGH"
 		(at 101.6 69.85 270)
 		(effects
@@
 		)
 	)
-	(label "B_HIGH"
+	(label "A_LOW"
 		(at 111.76 49.53 0)
 		(effects
@@
 		)
 	)
-	(label "A_LOW"
+	(label "B_LOW"
 		(at 111.76 59.69 0)
 		(effects
@@
 		)
 	)
-	(label "FBB"
+	(label "FBC"
 		(at 91.44 69.85 270)
 		(effects
@@
 		)
 	)
-	(label "FBC"
+	(label "FBB"
 		(at 93.98 69.85 270)
 		(effects
@@
 		)
 	)
+	(label "FBA"
+		(at 96.52 31.75 90)
+		(effects
+			(font
+				(size 1.27 1.27)
+			)
+			(justify left bottom)
+		)
+	)
 	(label "FBCOMMON"
 		(at 226.06 31.75 180)
@@
 		(dnp no)
 		(property "Reference" "R7"
-			(at 95.504 24.13 0)
+			(at 87.63 24.13 0)
 			(show_name no)
 			(do_not_autoplace no)
@@
 		)
 		(property "Value" "220R"
-			(at 95.504 26.67 0)
+			(at 87.63 26.67 0)
 			(show_name no)
 			(do_not_autoplace no)

Commit message: good placement 1
Parts:
- removed TP48: MOTORA, TestPoint:TestPoint_Pad_D1.0mm, symbol Connector:TestPoint
- removed TP52: MOTORB, TestPoint:TestPoint_Pad_D1.0mm, symbol Connector:TestPoint
- removed TP56: MOTORC, TestPoint:TestPoint_Pad_D1.0mm, symbol Connector:TestPoint

Commit message: something
Connections:
- net FBC: now also U5.9 (PA3); no longer U5.10 (PA4)
Changed lines of the file:
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@@
+	)
+	(no_connect
+		(at 91.44 69.85)
 	)
 	(no_connect
@@
 	)
 	(no_connect
-		(at 88.9 69.85)
-	)
-	(no_connect
 		(at 58.42 100.33)
 	)
@@
 		)
 	)
+	(label "FBC"
+		(at 88.9 69.85 270)
+		(effects
+			(font
+				(size 1.27 1.27)
+			)
+			(justify right bottom)
+		)
+	)
 	(label "GATE_A_HIGH"
 		(at 58.42 105.41 180)
@@
 		)
 	)
-	(label "FBC"
-		(at 91.44 69.85 270)
-		(effects
-			(font
-				(size 1.27 1.27)
-			)
-			(justify right bottom)
-		)
-	)
